Commit message: commit without kuka implementation

File: kuka_iiwa_support/urdf/kuka_iiwa_ctrl.xacro (robot description, xacro)
@@ -4,6 +4,6 @@
   <xacro:include filename="$(find kuka_iiwa_support)/urdf/kuka_iiwa_macro_ctrl.xacro"/>
   <xacro:arg name="robot_name" default="iiwa"/>
-	<link name="world"/>
-  <xacro:iiwa7 robot_name="$(arg robot_name)" parent="world">
+	<link name="base"/>
+  <xacro:iiwa7 robot_name="$(arg robot_name)" parent="base">
     <origin xyz="0 0 0" rpy="0 0 0" />
   </xacro:iiwa7>

File: turtlebot3_description/urdf/turtlebot3_burger.urdf.xacro (robot description, xacro)
@@ -149,5 +149,5 @@
   </link>
   <!--LASER SENSOR-->
-  <gazebo reference="base_footprint">
+  <gazebo reference="base_scan">
         <sensor type="ray" name="laser">
         <pose>0 0 0.1 0 0 0</pose>
@@ -180,5 +180,5 @@
         <plugin name="gazebo_ros_head_hokuyo_controller" filename="libgazebo_ros_laser.so">
           <topicName>/laser/scan</topicName>
-          <frameName>base_footprint</frameName>
+          <frameName>base_scan</frameName>
         </plugin>
       </sensor>

Commit message: last update working kuka (aruco_ros)

File: kuka_iiwa_support/urdf/kuka_iiwa_ctrl.xacro (robot description, xacro)
@@ -3,7 +3,8 @@
   <xacro:include filename="$(find kuka_iiwa_support)/urdf/utilities.xacro" />
   <xacro:include filename="$(find kuka_iiwa_support)/urdf/kuka_iiwa_macro_ctrl.xacro"/>
+  <xacro:include filename="$(find kuka_iiwa_support)/urdf/materials.xacro"/>
   <xacro:arg name="robot_name" default="iiwa"/>
-	<link name="base"/>
-  <xacro:iiwa7 robot_name="$(arg robot_name)" parent="base">
+	<link name="world"/>
+  <xacro:iiwa7 robot_name="$(arg robot_name)" parent="world">
     <origin xyz="0 0 0" rpy="0 0 0" />
   </xacro:iiwa7>

File: kuka_iiwa_support/urdf/kuka_iiwa_macro_ctrl.xacro (robot description, xacro)
@@ -261,4 +261,10 @@
       </collision>
     </link>
+    <joint name="camera_joint" type="fixed">
+    <parent link="${robot_name}_link_7"/>
+    <child link="camera_link"/>
+    <origin xyz="0 0 0.16" rpy="0 0 0"/>
+  </joint>
+  <link name="camera_link"/>
     <joint name="${robot_name}_joint_ee" type="fixed">
       <parent link="${robot_name}_link_7"/>
@@ -303,4 +309,41 @@
       <material>Gazebo/Grey</material>
 		</gazebo>
+    <!-- CAMERA SENSOR -->
+<gazebo reference="camera_link">
+    <sensor type="camera" name="camera">
+      <update_rate>30.0</update_rate>
+      <camera>
+        <horizontal_fov>1.3962634</horizontal_fov>
+        <image>
+          <width>800</width>
+          <height>600</height>
+          <format>R8G8B8</format>
+        </image>
+        <clip>
+          <near>0.02</near>
+          <far>30</far>
+        </clip>
+        <noise>
+          <type>gaussian</type>
+          <mean>0.0</mean>
+          <stddev>0.007</stddev>
+        </noise>
+      </camera>
+      <plugin name="camera_controller" filename="libgazebo_ros_camera.so">
+        <alwaysOn>true</alwaysOn>
+        <updateRate>0.0</updateRate>
+        <cameraName>camera</cameraName>
+        <imageTopicName>/kuka_iiwa/camera/image_raw</imageTopicName>
+        <cameraInfoTopicName>/kuka_iiwa/camera/camera_info</cameraInfoTopicName>
+        <frameName>camera_link</frameName>
+        <hackBaseline>0.07</hackBaseline>
+        <distortionK1>0.0</distortionK1>
+        <distortionK2>0.0</distortionK2>
+        <distortionK3>0.0</distortionK3>
+        <distortionT1>0.0</distortionT1>
+        <distortionT2>0.0</distortionT2>
+      </plugin>
+    </sensor>
+  </gazebo>
   </xacro:macro>
 </robot>
